File: SlyRaccoon/SlyRaccoon.kicad_sch (KiCad schematic)
At the start: 0 parts

Commit message: Start of schematic
- Matrix start
- MCU
- RGB Underglow
Parts:
- added D1, D10, D11, D12, D13, D14, D15, D16, D17, D18, D19, D2, D20, D21, D22, D23, D24, D3, D4, D5, D6, D7, D8, D9: 1N4148, Diode_THT:D_DO-35_SOD27_P7.62mm_Horizontal, symbol Diode:1N4148
- added D25, D26, D27, D28, D29, D30, D31, D32, D33, D34: SK6812, LED_SMD:LED_SK6812_PLCC4_5.0x5.0mm_P3.2mm, symbol LED:SK6812
- added SW1, SW10, SW11, SW12, SW13, SW14, SW15, SW16, SW17, SW18, SW19, SW2, SW20, SW21, SW22, SW23, SW3, SW4, SW5, SW6, SW7, SW8, SW9: SW_Push, Keebio:Kailh-PG1350-1u-NoLED, symbol Switch:SW_Push
- added SW24: SW_Push, Keebio:Kailh-PG1350-2u-NoLED, symbol Switch:SW_Push
- added U1: Elite-Pi, Keebio:Elite-C-castellated-29pin-holes, symbol SlyRaccoon:Elite-Pi
Connections:
- new net: D9.1 (K), SW8.1
- new net: D7.1 (K), SW4.1
- new net: D10.1 (K), SW5.1
- new net: D31.4 (DOUT), D32.2 (DIN)
- new net: D32.4 (DOUT), D33.2 (DIN)
- new net: D2.1 (K), SW2.1
- new net: D24.1 (K), SW24.1
- new net: D33.4 (DOUT), D34.2 (DIN)
- new net: D21.1 (K), SW20.1
- new net: D16.1 (K), SW14.1
- new net: D17.1 (K), SW15.1
- new net: D15.1 (K), SW12.1
- new net: D12.1 (K), SW10.1
- new net: D27.4 (DOUT), D28.2 (DIN)
- new net: D28.4 (DOUT), D29.2 (DIN)
- new net: D26.4 (DOUT), D27.2 (DIN)
- new net: D22.1 (K), SW22.1
- new net: D4.1 (K), SW13.1
- new net: D6.1 (K), SW21.1
- new net: D23.1 (K), SW23.1
- new net: D1.1 (K), SW1.1
- new net: D30.4 (DOUT), D31.2 (DIN)
- new net: D5.1 (K), SW17.1
- new net: D13.1 (K), SW6.1
- new net: D8.1 (K), SW7.1
- new net: D18.1 (K), SW16.1
- new net: D11.1 (K), SW9.1
- new net: D29.4 (DOUT), D30.2 (DIN)
- new net: D25.4 (DOUT), D26.2 (DIN)
- new net: D20.1 (K), SW19.1
- new net: D14.1 (K), SW11.1
- new net: D3.1 (K), SW3.1
- new net: D19.1 (K), SW18.1
- new net COL1: SW1.2, SW4.2, SW7.2, SW8.2, U1.9 (6/D6)
- new net COL2: SW10.2, SW2.2, SW5.2, SW9.2, U1.10 (7/D7)
- new net COL3: SW11.2, SW12.2, SW3.2, SW6.2, U1.11 (8/D8)
- new net COL4: SW13.2, SW14.2, SW15.2, SW16.2, U1.12 (9/D9)
- new net COL5: SW17.2, SW18.2, SW19.2, SW20.2, U1.13 (10/D21)
- new net COL6: SW21.2, SW22.2, SW23.2, SW24.2, U1.14 (16/D23)
- new net GND: D25.1 (VSS), D26.1 (VSS), D27.1 (VSS), D28.1 (VSS), D29.1 (VSS), D30.1 (VSS), D31.1 (VSS), D32.1 (VSS), D33.1 (VSS), D34.1 (VSS), U1.23 (GND), U1.3 (GND), U1.4 (GND)
- new net RGB: D25.2 (DIN), U1.15 (14/D20)
- new net ROW1: D1.2 (A), D2.2 (A), D3.2 (A), D4.2 (A), D5.2 (A), D6.2 (A), U1.5 (2/D2)
- new net ROW2: D10.2 (A), D13.2 (A), D16.2 (A), D19.2 (A), D22.2 (A), D7.2 (A), U1.6 (3/D3)
- new net ROW3: D11.2 (A), D14.2 (A), D17.2 (A), D20.2 (A), D23.2 (A), D8.2 (A), U1.7 (4/D4)
- new net ROW4: D12.2 (A), D15.2 (A), D18.2 (A), D21.2 (A), D24.2 (A), D9.2 (A), U1.8 (5/D5)
- new net RX: U1.2 (RX0/D1)
- new net TX: U1.1 (TX0/DO)
- no-connect marks 0 -> 2
Other:
- note added: "Matrix"
- note added: "RGB Underglow"
